File: 01_Logger/02_Modular_Logger/01_Electronics/02_Adapter/Analog-Adapter/Interface_Analog.kicad_sch (KiCad schematic)
At the start: 10 parts, among them IC301 TXB0104PW, K301 SSM3K127TU, X301 Molex Nano-Fit 105314-1*114

Commit message: Analog-Interfaceboard V0.2
Parts:
- C301, C302: eurocircuits_MPN (none) -> GPC0603104
- K301: eurocircuits_MPN (none) -> BSH105,215
- R303: now not fitted
- R304: value 0 -> 0R; eurocircuits_MPN (none) -> MCWR06X000 PTL
- X301: eurocircuits_MPN (none) -> 105314-1114
Connections:
- net GND: now also K301.2; no longer K301.3
- net Sensor_Lowside_Switch: now also K301.1; no longer K301.2
- net at X301.1 (Pin_1): now also K301.3; no longer K301.1
