File: 01_Logger/02_Modular_Logger/01_Electronics/02_Adapter/Analog-Adapter/MCU.kicad_sch (KiCad schematic)
At the start: 22 parts, among them IC201 MSP430FR2673, SW201 SKRKAEE020, SW202 A6H-8101, X201 ESQ-104-14-G-D, X202 Conn_02x03_Counter_Clockwise, X203 Conn_01x03, Y201 9HT11-32.768KDZF-T

Commit message: Analog-Interfaceboard V0.2
Parts:
- added C1: 100uF, Capacitor_SMD:C_0805_2012Metric_Pad1.18x1.45mm_HandSolder, symbol Device:C
- C201: eurocircuits_MPN (none) -> CL10B102KB8NNNC
- C202, C206: eurocircuits_MPN (none) -> CL10A105KB8NNNC
- C203, C204: eurocircuits_MPN (none) -> CL10C200JB8NNNC
- C205: eurocircuits_MPN (none) -> GPC0603104
- C207: eurocircuits_MPN (none) -> CL10A475KP8NNNC
- H201, H202, H203, H204, R203, R204: now not fitted
- IC201: eurocircuits_MPN (none) -> MSP430FR2673TRHBR
- R201: eurocircuits_MPN (none) -> RC0603FR-0747KL
- R202: eurocircuits_MPN (none) -> MCWR06X3300FTL
- SW201: eurocircuits_MPN (none) -> SKRKAEE020
- SW202: eurocircuits_MPN (none) -> A6H-8101
- X201: eurocircuits_MPN (none) -> ESQ-104-13-G-D
- X202: eurocircuits_MPN (none) -> PRT-12807
- X203: eurocircuits_MPN (none) -> 61300311121
- Y201: value 9HT11-32.768KDZF-T -> 9HT11-32.768KDZF-T; eurocircuits_MPN (none) -> 9HT11-32.768KDZF-T
Connections:
- net +3V3: now also C1.1
- net GND: now also C1.2
