File: 01_Logger/02_Modular_Logger/01_Electronics/01_Main_Unit/01_main_unit_MCI/Battery_Charger.kicad_sch (KiCad schematic)
At the start: 52 parts, among them IC501 BQ24618, J501 Conn_01x02, J502 Conn_01x02_Female, K501 SISH101DN-T1-GE3, K502 SISH101DN-T1-GE3, K503 SiS412DN, K504 SiS412DN, K505 SISH101DN-T1-GE3

Commit message: Main_Unit Update
Parts:
- C501: eurocircuits_MPN (none) -> KCM55WR7YA476MH01K
- C502, C503, C505, C506, C507, C511, C513, C514, C515: eurocircuits_MPN (none) -> 885012206095
- C504: eurocircuits_MPN (none) -> CL10A105KO8NNNC
- C508: eurocircuits_MPN (none) -> CL10B333KB8NNNC
- C509, C517: eurocircuits_MPN (none) -> EDK476M025A9GAA
- C510, C512: eurocircuits_MPN (none) -> CL10A105KB8NNNC
- C516, C518: eurocircuits_MPN (none) -> EDK226M035A9DAA
- C519: eurocircuits_MPN (none) -> 885012006053
- D501: eurocircuits_MPN (none) -> BAT54WX-TP
- IC501: eurocircuits_MPN (none) -> BQ24618RGET
- J501: eurocircuits_MPN (none) -> 43650-0215
- J502: eurocircuits_MPN (none) -> 53047-0210
- K501, K502, K505: eurocircuits_MPN (none) -> SI7101DN-T1-GE3
- K503, K504: eurocircuits_MPN (none) -> SIS412DN-T1-GE3
- L501: eurocircuits_MPN (none) -> SRP1245C-3R3M
- R501, R511: value 100 -> 100R; eurocircuits_MPN (none) -> MCWR06X1000FTL
- R502, R507: eurocircuits_MPN (none) -> MCWR06X1002FTL
- R503: eurocircuits_MPN (none) -> RP0603BRD075K76L
- R504: eurocircuits_MPN (none) -> RC0603FR-079K1L
- R505: eurocircuits_MPN (none) -> RC0603FR-07430KL
- R506, R510, R520: eurocircuits_MPN (none) -> MCWR06X1003FTL
- R508: eurocircuits_MPN (none) -> CPF0603B232KE1
- R509: eurocircuits_MPN (none) -> GPR060333K
- R512, R519: eurocircuits_MPN (none) -> MCWR06X1001FTL
- R513: value 0 -> 0R; eurocircuits_MPN (none) -> GPR06030R
- R514, R515, R516, R523: eurocircuits_MPN (none) -> ERA-3AEB4992V
- R517, R521: eurocircuits_MPN (none) -> PCS2512DR0100ET
- R518: value 10 -> 10R; eurocircuits_MPN (none) -> GPR060310R
- R522: eurocircuits_MPN (none) -> CRCW0603357KFKEA
