File: 01_Logger/02_Modular_Logger/01_Electronics/01_Main_Unit/01_main_unit_MCI/MPU.kicad_sch (KiCad schematic)
At the start: 34 parts, among them J1 Conn_01x02, J2 Conn_01x04_Pin, J3 Conn_01x04_Pin, J301 Conn_01x02, J302 Conn_02x04_Counter_Clockwise, J304 Conn_02x02_Odd_Even, SW301 SW_Push, U301 MAX16125WTEG00+T, U302 ESP32-S3-WROOM-1U, U303 DS3231MZ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

Commit message: Main_Unit Update
Parts:
- removed J1: Conn_01x02, Connector_Molex:Molex_PicoBlade_53047-0210_1x02_P1.25mm_Vertical, symbol Connector_Generic:Conn_01x02
- removed J2, J3: Conn_01x04_Pin, Connector_Molex:Molex_PicoBlade_53047-0410_1x04_P1.25mm_Vertical, symbol Connector:Conn_01x04_Pin
- removed R1, R2: 0R, Resistor_SMD:R_0603_1608Metric, symbol Device:R
- added H301, H302, H304, H306: MountingHole, MountingHole:MountingHole_3.2mm_M3_ISO7380, symbol Mechanical:MountingHole
- added J303: Conn_01x02, Connector_Molex:Molex_PicoBlade_53047-0210_1x02_P1.25mm_Vertical, symbol Connector_Generic:Conn_01x02
- added Q301: BSS138, Package_TO_SOT_SMD:SOT-23, symbol Transistor_FET:BSS138
- added R307: 75, Resistor_SMD:R_0603_1608Metric, symbol Device:R
- added R703: 1M, Resistor_SMD:R_0603_1608Metric, symbol Device:R
- added TP301, TP302: TestPoint, TestPoint:TestPoint_Pad_D1.0mm, symbol Connector:TestPoint
- C301, C302: eurocircuits_MPN CL10C200JB8NNNC -> (none)
- C303, C304, C305: eurocircuits_MPN 885012206095 -> (none)
- J301: eurocircuits_MPN 53047-0210 -> (none)
- J302: now fitted
- J304: eurocircuits_MPN 61300421121 -> (none)
- R301: value 470k -> 100k; eurocircuits_MPN GPR0603470K -> (none)
- R302, R303, R304, R305, R308, R309, R310: eurocircuits_MPN MCWR06X1002FTL -> (none)
- R306: value 68R -> 47k; eurocircuits_MPN GPR060368R -> (none)
- SW301: eurocircuits_MPN B3U-1000P -> (none)
- U301: eurocircuits_MPN MAX16125WTEG00+T -> (none)
- U302: eurocircuits_MPN ESP32-S3-WROOM-1U-N16R8 -> (none)
- U303: eurocircuits_MPN DS3231MZ+ -> (none)
- Y301: eurocircuits_MPN 9HT11-32.768KDZF-T -> (none)
Connections:
- net +3V3: now also J303.1 (Pin_1)
- net GND: now also Q301.2 (S), R703.2
- net I2C_SMBus_SCL: now also TP301.1
- net I2C_SMBus_SDA: now also TP302.1
- net RTC_INTERRUPT: now also U302.34 (IO41); no longer U302.21 (IO13)
- net at R306.2: now also Q301.1 (G)
- net LED_ROT renamed LED_STATUS
- net LED_STATUS: now also R703.1
- new net: J303.2 (Pin_2), R307.1
- new net: Q301.3 (D), R307.2
Other:
- note added: "100k at SEL => 5s delay"
- note added: "LED HLMP-EG1B-Z10DD Vf = 1.9 V If = 20mA 75 Ohm Vorwiderstand -> 18.67mA LED per Stecker absetzen!?"
- note removed: "470k at SEL => 23,5s delay"
