File: 01_Logger/02_Modular_Logger/01_Electronics/01_Main_Unit/01_main_unit_MCI/bms.kicad_sch (KiCad schematic)
At the start: 54 parts, among them IC801 BQ40Z80, J801 Conn_01x02_Male, J802 Conn_01x05_Male, J803 Conn_01x05_Female, K801 2N7002KW, K802 CSD18540Q5B, K803 DMP6023LSS-13, K804 CSD18540Q5B, SW801 SW_Push

Commit message: Main_Unit Update
Parts:
- C801, C802, C806, C807, C809, C812, C813, C815, C816, C817, C818: eurocircuits_MPN (none) -> 885012206095
- C803: eurocircuits_MPN (none) -> 885012206089
- C804, C805, C810, C814: eurocircuits_MPN (none) -> 885012006057
- C808: eurocircuits_MPN (none) -> C1812C225K1RACTU
- C811: eurocircuits_MPN (none) -> MCMT18N101F101CT
- D801, D803: eurocircuits_MPN (none) -> SS1H10-E3/61T
- D802: eurocircuits_MPN (none) -> MMSZ5246B-7-F
- F801: eurocircuits_MPN (none) -> SF-1206S1200R-2
- IC801: eurocircuits_MPN (none) -> BQ40Z80RSMT
- J801: eurocircuits_MPN (none) -> 53047-0210
- J802: eurocircuits_MPN (none) -> 43650-0515
- J803: now not fitted
- K801: eurocircuits_MPN (none) -> 2N7002KW
- K802, K804: eurocircuits_MPN (none) -> CSD18540Q5B
- K803: eurocircuits_MPN (none) -> DMP6023LSS-13
- R801: eurocircuits_MPN (none) -> MCWR06X1101FTL
- R802, R809: eurocircuits_MPN (none) -> MCWR06X1002FTL
- R803, R807, R810: eurocircuits_MPN (none) -> RC0603FR-0710ML
- R804: eurocircuits_MPN (none) -> CPF0603F4K87C1
- R805: value 510 -> 510R; eurocircuits_MPN (none) -> RC0603FR-07510RL
- R806: value 51 -> 51R; eurocircuits_MPN (none) -> GPR060351R
- R808: eurocircuits_MPN (none) -> MCWR06X1001FTL
- R811: eurocircuits_MPN (none) -> 356047RJT
- R812, R814, R815: value 100 -> 100R; eurocircuits_MPN (none) -> MCWR06X1000FTL
- R813: eurocircuits_MPN (none) -> WSLP12061L000FEA
- R816, R817, R818, R819: value 499 -> 499R; eurocircuits_MPN (none) -> ERJ3EKF4990V
- SW801: eurocircuits_MPN (none) -> B3U-1000P
