File: 01_Logger/02_Modular_Logger/01_Electronics/01_Main_Unit/01_main_unit_MCI/main_unit.kicad_sch (KiCad schematic)
At the start: 1 part, among them J102 FTS-107-01-F-D

Commit message: Main_Unit Update
Parts:
- removed J102: FTS-107-01-F-D, Connector_PinHeader_1.27mm:PinHeader_2x07_P1.27mm_Vertical, symbol Connector_Generic:Conn_02x07_Counter_Clockwise
- added J101: SFMC-107-01-L-D, Connector_PinSocket_1.27mm:PinSocket_2x07_P1.27mm_Vertical, symbol Connector_Generic:Conn_02x07_Counter_Clockwise
Connections:
- net +12V: now also J101.12 (Pin_12)
- net +3V3: now also J101.10 (Pin_10)
- net +5V: now also J101.11 (Pin_11)
- net GND: now also J101.7 (Pin_7), J101.8 (Pin_8)
- new net power/Charge_Enable: J101.3 (Pin_3)
- new net power/ENABLE_12V: J101.2 (Pin_2)
- new net power/ENABLE_5V: J101.1 (Pin_1)
- new net power/I2C_SMBus_SCL: J101.14 (Pin_14)
- new net power/I2C_SMBus_SDA: J101.13 (Pin_13)
- new net power/~{PG}: J101.4 (Pin_4)
- new net power/~{STAT1}: J101.6 (Pin_6)
- new net power/~{STAT2}: J101.5 (Pin_5)
Other:
- removed sheet MPU
- removed sheet memory
- added sheet power (power.kicad_sch)
