File: 01_Logger/02_Modular_Logger/01_Electronics/01_Main_Unit/01_main_unit_MCI/memory.kicad_sch (KiCad schematic)
At the start: 3 parts, among them J701 Micro_SD_Card_Det

Commit message: Main_Unit Update
Parts:
- J701: eurocircuits_MPN 693071020811 -> (none)
- R701, R702: eurocircuits_MPN MCWR06X1002FTL -> (none)
Changed lines of the file:
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@@
-			)
-		)
-		(property "eurocircuits_MPN" "693071020811"
-			(at 175.26 86.36 0)
-			(effects
-				(font
-					(size 1.27 1.27)
-				)
-				(hide yes)
 			)
 		)
@@
 			)
 		)
-		(property "eurocircuits_MPN" "MCWR06X1002FTL"
-			(at 124.46 97.79 0)
-			(effects
-				(font
-					(size 1.27 1.27)
-				)
-				(hide yes)
-			)
-		)
 		(pin "1"
 		)
@@
 			(effects
 				(font
-					(size 1.27 1.27)
-				)
-				(hide yes)
-			)
-		)
-		(property "eurocircuits_MPN" "MCWR06X1002FTL"
-			(at 151.13 114.3 90)
-			(effects
-				(font
