File: 01_Logger/02_Modular_Logger/01_Electronics/01_Main_Unit/01_main_unit_MCI/voltage_regulators.kicad_sch (KiCad schematic)
At the start: 22 parts, among them Q601 BSS123, Q602 IRLML5203TRPBF, Q603 BSS123, Q604 IRLML5203TRPBF, U601 SPBW06F-12, U602 OKI-78SR-3.3_1.5-W36-C, U603 OKI-78SR-5_1.5-W36-C

Commit message: Main_Unit Update
Parts:
- C601: eurocircuits_MPN (none) -> 860020672010
- C602, C603: eurocircuits_MPN (none) -> C2012X5R1V226M125AC
- C604: eurocircuits_MPN (none) -> CC1206JKNPODBN151
- C605, C606: eurocircuits_MPN (none) -> GRM21BR61A476ME15L
- L601: eurocircuits_MPN (none) -> CC453232A-100KL
- Q601, Q603: eurocircuits_MPN (none) -> BSS123
- Q602, Q604: eurocircuits_MPN (none) -> IRLML5203TRPBF
- R601, R605: eurocircuits_MPN (none) -> MCWR06X2701FTL
- R602, R606: eurocircuits_MPN (none) -> RC0603FR-0747KL
- R603, R607: eurocircuits_MPN (none) -> RC0603FR-07680KL
- R604, R608: eurocircuits_MPN (none) -> MCWR06X1001FTL
- U601: eurocircuits_MPN (none) -> SPBW06F-12
- U602: eurocircuits_MPN (none) -> TSR 1-2433E
- U603: eurocircuits_MPN (none) -> TSR 1-2450
Changed lines of the file:
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@@
+			)
+		)
+		(property "eurocircuits_MPN" "IRLML5203TRPBF"
+			(at 139.7 78.74 90)
+			(effects
+				(font
+					(size 1.27 1.27)
+				)
+				(hide yes)
 			)
 		)
@@
 			)
 		)
+		(property "eurocircuits_MPN" "MCWR06X2701FTL"
+			(at 93.98 106.68 0)
+			(effects
+				(font
+					(size 1.27 1.27)
+				)
+				(hide yes)
+			)
+		)
 		(pin "1"
 		)
@@
 			)
 		)
+		(property "eurocircuits_MPN" "860020672010"
+			(at 125.73 142.24 0)
+			(effects
+				(font
+					(size 1.27 1.27)
+				)
+				(hide yes)
+			)
+		)
 		(pin "1"
 		)
@@
 			)
 		)
+		(property "eurocircuits_MPN" "MCWR06X1001FTL"
+			(at 81.28 153.67 90)
+			(effects
+				(font
+					(size 1.27 1.27)
+				)
+				(hide yes)
+			)
+		)
 		(pin "1"
 		)
@@
 			)
 		)
+		(property "eurocircuits_MPN" "MCWR06X1001FTL"
+			(at 129.54 93.98 90)
+			(effects
+				(font
+					(size 1.27 1.27)
+				)
+				(hide yes)
+			)
+		)
 		(pin "1"
 		)
@@
 			)
 		)
+		(property "eurocircuits_MPN" "BSS123"
+			(at 68.58 160.02 0)
+			(effects
+				(font
+					(size 1.27 1.27)
+				)
+				(hide yes)
+			)
+		)
 		(pin "1"
 		)
@@
 			)
 		)
+		(property "eurocircuits_MPN" "BSS123"
+			(at 116.84 100.33 0)
+			(effects
+				(font
+					(size 1.27 1.27)
+				)
+				(hide yes)
+			)
+		)
 		(pin "1"
 		)
@@
 			)
 		)
+		(property "eurocircuits_MPN" "GRM21BR61A476ME15L"
+			(at 195.58 31.75 0)
+			(effects
+				(font
+					(size 1.27 1.27)
+				)
+				(hide yes)
+			)
+		)
 		(pin "1"
 		)
@@
 			)
 		)
+		(property "eurocircuits_MPN" "RC0603FR-0747KL"
+			(at 53.34 160.02 90)
+			(effects
+				(font
+					(size 1.27 1.27)
+				)
+				(hide yes)
+			)
+		)
 		(pin "1"
 		)
@@
 			)
 		)
+		(property "eurocircuits_MPN" "SPBW06F-12"
+			(at 167.64 140.97 0)
+			(effects
+				(font
+					(size 1.27 1.27)
+				)
+				(hide yes)
+			)
+		)
 		(pin "1"
 		)
@@
 			)
 		)
+		(property "eurocircuits_MPN" "MCWR06X2701FTL"
+			(at 45.72 166.37 0)
+			(effects
+				(font
+					(size 1.27 1.27)
+				)
+				(hide yes)
+			)
+		)
 		(pin "1"
 		)
@@
 			)
 		)
+		(property "eurocircuits_MPN" "RC0603FR-0747KL"
+			(at 101.6 100.33 90)
+			(effects
+				(font
+					(size 1.27 1.27)
+				)
+				(hide yes)
+			)
+		)
 		(pin "1"
 		)
@@
 			)
 		)
+		(property "eurocircuits_MPN" "RC0603FR-07680KL"
+			(at 125.73 82.55 0)
+			(effects
+				(font
+					(size 1.27 1.27)
+				)
+				(hide yes)
+			)
+		)
 		(pin "1"
 		)
@@
 			)
 		)
+		(property "eurocircuits_MPN" "TSR 1-2450"
+			(at 180.34 76.2 0)
+			(effects
+				(font
+					(size 1.27 1.27)
+				)
+				(hide yes)
+			)
+		)
 		(pin "1"
 		)
@@
 			)
 		)
+		(property "eurocircuits_MPN" "TSR 1-2433E"
+			(at 180.34 25.4 0)
+			(effects
+				(font
+					(size 1.27 1.27)
+				)
+				(hide yes)
+			)
+		)
 		(pin "1"
 		)
@@
 			)
 		)
+		(property "eurocircuits_MPN" "GRM21BR61A476ME15L"
+			(at 195.58 82.55 0)
+			(effects
+				(font
+					(size 1.27 1.27)
+				)
+				(hide yes)
+			)
+		)
 		(pin "1"
 		)
@@
 			)
 		)
+		(property "eurocircuits_MPN" "C2012X5R1V226M125AC"
+			(at 165.1 82.55 0)
+			(effects
+				(font
+					(size 1.27 1.27)
+				)
+				(hide yes)
+			)
+		)
 		(pin "1"
 		)
@@
 			)
 		)
+		(property "eurocircuits_MPN" "RC0603FR-07680KL"
+			(at 77.47 142.24 0)
+			(effects
+				(font
+					(size 1.27 1.27)
+				)
+				(hide yes)
+			)
+		)
 		(pin "1"
 		)
@@
 		)
 		(property "Description" ""
+			(at 165.1 31.75 0)
+			(effects
+				(font
+					(size 1.27 1.27)
+				)
+				(hide yes)
+			)
+		)
+		(property "eurocircuits_MPN" "C2012X5R1V226M125AC"
 			(at 165.1 31.75 0)
 			(effects
@@
 			)
 		)
+		(property "eurocircuits_MPN" "IRLML5203TRPBF"
+			(at 91.44 138.43 90)
+			(effects
+				(font
+					(size 1.27 1.27)
+				)
+				(hide yes)
+			)
+		)
 		(pin "1"
 		)
@@
 			)
 		)
+		(property "eurocircuits_MPN" "CC1206JKNPODBN151"
+			(at 168.91 123.19 90)
+			(effects
+				(font
+					(size 1.27 1.27)
+				)
+				(hide yes)
+			)
+		)
 		(pin "1"
 		)
@@
 			(at 138.43 135.89 0)
 			(effects
+				(font
+					(size 1.27 1.27)
+				)
+				(hide yes)
+			)
+		)
+		(property "eurocircuits_MPN" "CC453232A-100KL"
+			(at 138.43 135.89 0)
+			(effects
