File: 01_Logger/02_Modular_Logger/01_Electronics/01_Main_Unit/01_main_unit_MCU/MPU.kicad_sch (KiCad schematic)
At the start: 35 parts, among them J301 Conn_01x02, J302 Conn_02x04_Counter_Clockwise, J303 Conn_01x02, J304 Conn_02x02_Odd_Even, Q301 BSS138, SW301 SW_Push, U301 MAX16125WTEG00+T, U302 ESP32-S3-WROOM-1U, U303 DS3231MZ, Y301 Crystal

Commit message: Main_Unit Update
Parts:
- removed J303: Conn_01x02, Connector_Molex:Molex_PicoBlade_53047-0210_1x02_P1.25mm_Vertical, symbol Connector_Generic:Conn_01x02
- removed Q301: BSS138, Package_TO_SOT_SMD:SOT-23, symbol Transistor_FET:BSS138
- removed R307: 75, Resistor_SMD:R_0603_1608Metric, symbol Device:R
- removed R703: 1M, Resistor_SMD:R_0603_1608Metric, symbol Device:R
- removed TP301, TP302: TestPoint, TestPoint:TestPoint_Pad_D1.0mm, symbol Connector:TestPoint
- added J1: Conn_01x02, Connector_Molex:Molex_PicoBlade_53047-0210_1x02_P1.25mm_Vertical, symbol Connector_Generic:Conn_01x02
- added J2, J3: Conn_01x04_Pin, Connector_Molex:Molex_PicoBlade_53047-0410_1x04_P1.25mm_Vertical, symbol Connector:Conn_01x04_Pin
- added R1, R2: 0R, Resistor_SMD:R_0603_1608Metric, symbol Device:R
- R301: value 100k -> 470k; eurocircuits_MPN MCWR06X1003FTL -> GPR0603470K
- R306: value 47k -> 68R; eurocircuits_MPN RC0603FR-0747KL -> GPR060368R
Connections:
- net +3V3: now also J3.4 (Pin_4)
- net GND: now also J1.2 (Pin_2), J2.4 (Pin_4), J3.1 (Pin_1)
- net I2C_SMBus_SCL: now also J3.2 (Pin_2)
- net I2C_SMBus_SDA: now also J3.3 (Pin_3)
- net RTC_INTERRUPT: now also U302.21 (IO13); no longer U302.34 (IO41)
- net at U302.15 (IO3): now also J1.1 (Pin_1)
- net at U302.29 (IO36): now also R1.2
- net at U302.30 (IO37): now also R2.2
- net at R306.2: now also J2.2 (Pin_2)
- net LED_STATUS renamed LED_ROT
- new net: J2.1 (Pin_1), R2.1
- new net: J2.3 (Pin_3), R1.1
Other:
- note added: "470k at SEL => 23,5s delay"
- note removed: "100k at SEL => 5s delay"
- note removed: "LED HLMP-EG1B-Z10DD Vf = 1.9 V If = 20mA 75 Ohm Vorwiderstand -> 18.67mA LED per Stecker absetzen!?"
