File: 01_Logger/02_Modular_Logger/01_Electronics/01_Main_Unit/01_main_unit_MCU/main_unit.kicad_pcb (KiCad board)
At the start: 4 copper layers, 54.9 x 27.4 mm, 35 parts, among them J102 FTS-107-01-F-D, J301 Conn_01x02, J302 Conn_02x04_Counter_Clockwise, J303 Conn_01x02, J304 Conn_02x02_Odd_Even, J701 Micro_SD_Card_Det, Q301 BSS138, SW301 SW_Push, U301 MAX16125WTEG00+T, U302 ESP32-S3-WROOM-1U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

Commit message: Main_Unit Update
Parts:
- removed J303: Conn_01x02, Connector_Molex:Molex_PicoBlade_53047-0210_1x02_P1.25mm_Vertical
- removed Q301: BSS138, Package_TO_SOT_SMD:SOT-23
- removed R307: 75, Resistor_SMD:R_0603_1608Metric
- removed R703: 1M, Resistor_SMD:R_0603_1608Metric
- removed TP301, TP302: TestPoint, TestPoint:TestPoint_Pad_D1.0mm
- added J1: Conn_01x02, Connector_Molex:Molex_PicoBlade_53047-0210_1x02_P1.25mm_Vertical, F.Cu at (209.8, 103.5)
- added J2: Conn_01x04_Pin, Connector_Molex:Molex_PicoBlade_53047-0410_1x04_P1.25mm_Vertical, F.Cu at (201.2, 103.5)
- added J3: Conn_01x04_Pin, Connector_Molex:Molex_PicoBlade_53047-0410_1x04_P1.25mm_Vertical, F.Cu at (206.3, 98.5)
- added R1: 0R, Resistor_SMD:R_0603_1608Metric, F.Cu at (195.4, 104.3)
- added R2: 0R, Resistor_SMD:R_0603_1608Metric, F.Cu at (197.7, 102.7)
- R301: value 100k -> 470k
- R306: value 47k -> 68R
- moved TP303 5.55 mm to (201.6, 98.5)
- moved R308 3.03 mm to (197.9, 98.3)
Connections:
- net /MPU/LED_STATUS renamed /MPU/LED_ROT
- U302 pad 21: unconnected-(U302-IO13-Pad21) -> /MPU/RTC_INTERRUPT
- U302 pad 34: /MPU/RTC_INTERRUPT -> unconnected-(U302-IO41-Pad34)
Routing:
- net unconnected-(J1-Pin_1-Pad1): track 0.00 -> 34.5 mm
- net /MPU/RTC_INTERRUPT: track 10.4 -> 26.8 mm, vias 0 -> 4
- net Net-(J2-Pin_3): track 0.00 -> 8.63 mm
- net Net-(J2-Pin_2): track 2.73 -> 9.73 mm
- net GND: track 43.4 -> 36.7 mm
- net unconnected-(R2-Pad2): track 0.00 -> 6.45 mm
- net /MPU/I2C_SMBus_SCL: track 83.5 -> 89.6 mm, vias 6 -> 7
- net unconnected-(R1-Pad2): track 0.00 -> 4.86 mm
- net Net-(Q301-D): track 4.44 -> 0.00 mm
- net Net-(J303-Pin_2): track 3.84 -> 0.00 mm
- net /MPU/I2C_SMBus_SDA: track 75.4 -> 78.8 mm
- net Net-(J2-Pin_1): track 0.00 -> 3.00 mm
- net /MPU/LED_ROT: track 18.8 -> 16.8 mm
Other:
- outline, holes or cut-outs redrawn
- board text added: "-"
- board text added: "------"
- board text added: "3V3"
- board text added: "BMS"
- board text added: "GND"
- board text added: "HyFiVe Logger-MPU-Board V0.5 08/2025"
- board text added: "RX"
- board text added: "SCL"
- board text added: "SDA"
- board text added: "TX"
- board text removed: "HyFiVe Logger-MPU-Board V0.4 06/2025"
- board text removed: "SDA SCL GND"
